Commit message: Update Robot.xacro

File: proyecto/urdf/Robot.xacro (robot description, xacro)
@@ -1,7 +1,7 @@
 <?xml version="1.0" ?>
 <robot name="Robot" xmlns:xacro="http://www.ros.org/wiki/xacro">
-<xacro:include filename="$(find Robot_description)/urdf/materials.xacro" />
-<xacro:include filename="$(find Robot_description)/urdf/Robot.trans" />
-<xacro:include filename="$(find Robot_description)/urdf/Robot.gazebo" />
+<xacro:include filename="$(find proyecto)/urdf/materials.xacro" />
+<xacro:include filename="$(find proyecto)/urdf/Robot.trans" />
+<xacro:include filename="$(find proyecto)/urdf/Robot.gazebo" />
 <link name="base_link">
   <inertial>
@@ -13,5 +13,5 @@
     <origin xyz="0 0 0" rpy="0 0 0"/>
     <geometry>
-      <mesh filename="package://Robot_description/meshes/base_link.stl" scale="0.001 0.001 0.001"/>
+      <mesh filename="package://proyecto/meshes/base_link.stl" scale="0.001 0.001 0.001"/>
     </geometry>
     <material name="silver"/>
@@ -20,5 +20,5 @@
     <origin xyz="0 0 0" rpy="0 0 0"/>
     <geometry>
-      <mesh filename="package://Robot_description/meshes/base_link.stl" scale="0.001 0.001 0.001"/>
+      <mesh filename="package://proyecto/meshes/base_link.stl" scale="0.001 0.001 0.001"/>
     </geometry>
   </collision>
@@ -33,5 +33,5 @@
     <origin xyz="0.011211 -2.022818 -0.91961" rpy="0 0 0"/>
     <geometry>
-      <mesh filename="package://Robot_description/meshes/placa_base_1.stl" scale="0.001 0.001 0.001"/>
+      <mesh filename="package://proyecto/meshes/placa_base_1.stl" scale="0.001 0.001 0.001"/>
     </geometry>
     <material name="silver"/>
@@ -40,5 +40,5 @@
     <origin xyz="0.011211 -2.022818 -0.91961" rpy="0 0 0"/>
     <geometry>
-      <mesh filename="package://Robot_description/meshes/placa_base_1.stl" scale="0.001 0.001 0.001"/>
+      <mesh filename="package://proyecto/meshes/placa_base_1.stl" scale="0.001 0.001 0.001"/>
     </geometry>
   </collision>
@@ -53,5 +53,5 @@
     <origin xyz="-0.397565 -0.568456 -0.317359" rpy="0 0 0"/>
     <geometry>
-      <mesh filename="package://Robot_description/meshes/base_r_1.stl" scale="0.001 0.001 0.001"/>
+      <mesh filename="package://proyecto/meshes/base_r_1.stl" scale="0.001 0.001 0.001"/>
     </geometry>
     <material name="silver"/>
@@ -60,5 +60,5 @@
     <origin xyz="-0.397565 -0.568456 -0.317359" rpy="0 0 0"/>
     <geometry>
-      <mesh filename="package://Robot_description/meshes/base_r_1.stl" scale="0.001 0.001 0.001"/>
+      <mesh filename="package://proyecto/meshes/base_r_1.stl" scale="0.001 0.001 0.001"/>
     </geometry>
   </collision>
@@ -73,5 +73,5 @@
     <origin xyz="-0.397565 -0.568456 -0.609359" rpy="0 0 0"/>
     <geometry>
-      <mesh filename="package://Robot_description/meshes/s_axis_1.stl" scale="0.001 0.001 0.001"/>
+      <mesh filename="package://proyecto/meshes/s_axis_1.stl" scale="0.001 0.001 0.001"/>
     </geometry>
     <material name="silver"/>
@@ -80,5 +80,5 @@
     <origin xyz="-0.397565 -0.568456 -0.609359" rpy="0 0 0"/>
     <geometry>
-      <mesh filename="package://Robot_description/meshes/s_axis_1.stl" scale="0.001 0.001 0.001"/>
+      <mesh filename="package://proyecto/meshes/s_axis_1.stl" scale="0.001 0.001 0.001"/>
     </geometry>
   </collision>
@@ -93,5 +93,5 @@
     <origin xyz="-1.137571 -0.490512 -0.757359" rpy="0 0 0"/>
     <geometry>
-      <mesh filename="package://Robot_description/meshes/l_axis_1.stl" scale="0.001 0.001 0.001"/>
+      <mesh filename="package://proyecto/meshes/l_axis_1.stl" scale="0.001 0.001 0.001"/>
     </geometry>
     <material name="silver"/>
@@ -100,5 +100,5 @@
     <origin xyz="-1.137571 -0.490512 -0.757359" rpy="0 0 0"/>
     <geometry>
-      <mesh filename="package://Robot_description/meshes/l_axis_1.stl" scale="0.001 0.001 0.001"/>
+      <mesh filename="package://proyecto/meshes/l_axis_1.stl" scale="0.001 0.001 0.001"/>
     </geometry>
   </collision>
@@ -113,5 +113,5 @@
     <origin xyz="-1.137534 -0.301512 -1.907359" rpy="0 0 0"/>
     <geometry>
-      <mesh filename="package://Robot_description/meshes/u_axis_1.stl" scale="0.001 0.001 0.001"/>
+      <mesh filename="package://proyecto/meshes/u_axis_1.stl" scale="0.001 0.001 0.001"/>
     </geometry>
     <material name="silver"/>
@@ -120,5 +120,5 @@
     <origin xyz="-1.137534 -0.301512 -1.907359" rpy="0 0 0"/>
     <geometry>
-      <mesh filename="package://Robot_description/meshes/u_axis_1.stl" scale="0.001 0.001 0.001"/>
+      <mesh filename="package://proyecto/meshes/u_axis_1.stl" scale="0.001 0.001 0.001"/>
     </geometry>
   </collision>
@@ -133,5 +133,5 @@
     <origin xyz="-2.166033 -0.568589 -2.157277" rpy="0 0 0"/>
     <geometry>
-      <mesh filename="package://Robot_description/meshes/r_axis_1.stl" scale="0.001 0.001 0.001"/>
+      <mesh filename="package://proyecto/meshes/r_axis_1.stl" scale="0.001 0.001 0.001"/>
     </geometry>
     <material name="silver"/>
@@ -140,5 +140,5 @@
     <origin xyz="-2.166033 -0.568589 -2.157277" rpy="0 0 0"/>
     <geometry>
-      <mesh filename="package://Robot_description/meshes/r_axis_1.stl" scale="0.001 0.001 0.001"/>
+      <mesh filename="package://proyecto/meshes/r_axis_1.stl" scale="0.001 0.001 0.001"/>
     </geometry>
   </collision>
@@ -153,5 +153,5 @@
     <origin xyz="-2.362546 -0.399739 -2.157247" rpy="0 0 0"/>
     <geometry>
-      <mesh filename="package://Robot_description/meshes/b_axis_1.stl" scale="0.001 0.001 0.001"/>
+      <mesh filename="package://proyecto/meshes/b_axis_1.stl" scale="0.001 0.001 0.001"/>
     </geometry>
     <material name="silver"/>
@@ -160,5 +160,5 @@
     <origin xyz="-2.362546 -0.399739 -2.157247" rpy="0 0 0"/>
     <geometry>
-      <mesh filename="package://Robot_description/meshes/b_axis_1.stl" scale="0.001 0.001 0.001"/>
+      <mesh filename="package://proyecto/meshes/b_axis_1.stl" scale="0.001 0.001 0.001"/>
     </geometry>
   </collision>
@@ -173,5 +173,5 @@
     <origin xyz="-2.582537 -0.527255 -2.157192" rpy="0 0 0"/>
     <geometry>
-      <mesh filename="package://Robot_description/meshes/t_axis_1.stl" scale="0.001 0.001 0.001"/>
+      <mesh filename="package://proyecto/meshes/t_axis_1.stl" scale="0.001 0.001 0.001"/>
     </geometry>
     <material name="silver"/>
@@ -180,5 +180,5 @@
     <origin xyz="-2.582537 -0.527255 -2.157192" rpy="0 0 0"/>
     <geometry>
-      <mesh filename="package://Robot_description/meshes/t_axis_1.stl" scale="0.001 0.001 0.001"/>
+      <mesh filename="package://proyecto/meshes/t_axis_1.stl" scale="0.001 0.001 0.001"/>
     </geometry>
   </collision>
@@ -193,5 +193,5 @@
     <origin xyz="-1.412434 -1.519454 -1.498385" rpy="0 0 0"/>
     <geometry>
-      <mesh filename="package://Robot_description/meshes/balancer_2_1.stl" scale="0.001 0.001 0.001"/>
+      <mesh filename="package://proyecto/meshes/balancer_2_1.stl" scale="0.001 0.001 0.001"/>
     </geometry>
     <material name="silver"/>
@@ -200,5 +200,5 @@
     <origin xyz="-1.412434 -1.519454 -1.498385" rpy="0 0 0"/>
     <geometry>
-      <mesh filename="package://Robot_description/meshes/balancer_2_1.stl" scale="0.001 0.001 0.001"/>
+      <mesh filename="package://proyecto/meshes/balancer_2_1.stl" scale="0.001 0.001 0.001"/>
     </geometry>
   </collision>
@@ -213,5 +213,5 @@
     <origin xyz="0.078722 -1.952822 -1.863697" rpy="0 0 0"/>
     <geometry>
-      <mesh filename="package://Robot_description/meshes/balancer_1_1.stl" scale="0.001 0.001 0.001"/>
+      <mesh filename="package://proyecto/meshes/balancer_1_1.stl" scale="0.001 0.001 0.001"/>
     </geometry>
     <material name="silver"/>
@@ -220,5 +220,5 @@
     <origin xyz="0.078722 -1.952822 -1.863697" rpy="0 0 0"/>
     <geometry>
-      <mesh filename="package://Robot_description/meshes/balancer_1_1.stl" scale="0.001 0.001 0.001"/>
+      <mesh filename="package://proyecto/meshes/balancer_1_1.stl" scale="0.001 0.001 0.001"/>
     </geometry>
   </collision>
